Commit message: Add cable guide and additional collision body to URDF/XACRO
Both objects allow better self collision avoidance.

File: iai_daisy_description/robots/daisy.urdf.xacro (robot description, xacro)
@@ -61,4 +61,57 @@
   <xacro:property name="right_arm_mounting_plate_x_offset" value="0.994" />
   <xacro:property name="right_arm_mounting_plate_y_offset" value="0.368" />
+  <!-- Gripper cable guide properties + macro === -->
+  <xacro:property name="gripper_side_cylinder_length" value="0.10" />
+  <xacro:property name="gripper_side_cylinder_radius" value="0.0175" /> <!-- 3.5 cm diameter -->
+  <xacro:property name="gripper_side_cylinder_y_offset" value="0.075" /> <!-- adjust to clear the mounting plate edge -->
+  <xacro:macro name="gripper_side_cylinder" params="parent prefix">
+    <link name="${prefix}_side_cylinder_link">
+      <visual>
+        <origin xyz="0 0 0" rpy="0 0 0"/>
+        <geometry>
+          <cylinder length="${gripper_side_cylinder_length}" radius="${gripper_side_cylinder_radius}"/>
+        </geometry>
+        <material name="grey"/>
+      </visual>
+      <collision>
+        <origin xyz="0 0 0" rpy="0 0 0"/>
+        <geometry>
+          <cylinder length="${gripper_side_cylinder_length}" radius="${gripper_side_cylinder_radius}"/>
+        </geometry>
+      </collision>
+    </link>
+    <joint name="${prefix}_side_cylinder_joint" type="fixed">
+      <parent link="${parent}"/>
+      <child link="${prefix}_side_cylinder_link"/>
+      <!-- offset in +Y of the parent frame; rpy=0 keeps the cylinder's
+           native Z-axis aligned with the parent's Z-axis -->
+      <origin xyz="0 ${gripper_side_cylinder_y_offset} -${gripper_side_cylinder_length/2 - 0.02}" rpy="0 0 0"/>
+    </joint>
+  </xacro:macro>
+    <!-- Gripper Wrist 2 collision === -->
+  <xacro:property name="gripper_collision_cylinder_length" value="0.005" />
+  <xacro:property name="gripper_collision_cylinder_radius" value="0.034" /> <!-- 7.2 cm diameter -->
+  <xacro:macro name="wrist_collision_cylinder_macro" params="parent prefix">
+    <link name="${prefix}_wrist_collision_cylinder_link">
+      <visual>
+        <origin xyz="0 0 0" rpy="0 0 0"/>
+        <geometry>
+          <cylinder length="${gripper_collision_cylinder_length}" radius="${gripper_collision_cylinder_radius}"/>
+        </geometry>
+        <material name="grey"/>
+      </visual>
+      <collision>
+        <origin xyz="0 0 0" rpy="0 0 0"/>
+        <geometry>
+          <cylinder length="${gripper_collision_cylinder_length}" radius="${gripper_collision_cylinder_radius}"/>
+        </geometry>
+      </collision>
+    </link>
+    <joint name="${prefix}_wrist_collision_cylinder_joint" type="fixed">
+      <parent link="${parent}"/>
+      <child link="${prefix}_wrist_collision_cylinder_link"/>
+      <origin xyz="0 -0.051 -0.0028" rpy="${pi/2} 0 0"/>
+    </joint>
+  </xacro:macro>
   <link name="map" />
   <joint name="table_joint" type="fixed">
@@ -110,5 +163,5 @@
   <link name="left_gripper_mounting_plate">
     <visual>
-      <origin xyz="0 0 0" rpy="0 0 ${pi/2}"/>
+      <origin xyz="0 0 0" rpy="${pi} 0 ${pi/2}"/>
       <geometry>
         <mesh filename="package://iai_daisy_description/meshes/FL-ISO50-WPG300_WITH_FILLET.stl" scale="0.001 0.001 0.001"/>
@@ -117,5 +170,5 @@
     </visual>
     <collision>
-      <origin xyz="0 0 0" rpy="0 0 ${pi/2}"/>
+      <origin xyz="0 0 0" rpy="${pi} 0 ${pi/2}"/>
       <geometry>
         <mesh filename="package://iai_daisy_description/meshes/FL-ISO50-WPG300_WITH_FILLET.stl" scale="0.001 0.001 0.001"/>
@@ -126,8 +179,11 @@
     <parent link="left_flange"/>
     <child link="left_gripper_mounting_plate"/>
-    <origin xyz="0 0 0.005" rpy="${pi/2} 0 ${pi/2}"/>
-  </joint>
+    <origin xyz="0.005 0 0" rpy="${pi/2} 0 ${pi/2}"/>
+  </joint>
+  <!-- === Cable guide on the left gripper === -->
+  <xacro:gripper_side_cylinder parent="left_gripper_mounting_plate" prefix="left_gripper" />
+  <xacro:wrist_collision_cylinder_macro parent="left_wrist_2_link" prefix="left_gripper" />
   <xacro:wsg_300_120_xacro parent="left_gripper_mounting_plate" name="left_gripper">
-    <origin xyz="0 0 0" rpy="0 0 -${pi/2}"/>
+    <origin xyz="0 0 0.005" rpy="0 0 -${pi/2}"/>
   </xacro:wsg_300_120_xacro>
   <joint name="right_arm_mounting_plate_joint" type="fixed">
@@ -160,5 +216,5 @@
   <link name="right_gripper_mounting_plate">
     <visual>
-      <origin xyz="0 0 0" rpy="0 0 ${pi/2}"/>
+      <origin xyz="0 0 0" rpy="${pi} 0 ${pi/2}"/>
       <geometry>
         <mesh filename="package://iai_daisy_description/meshes/FL-ISO50-WPG300_WITH_FILLET.stl" scale="0.001 0.001 0.001"/>
@@ -166,5 +222,5 @@
     </visual>
     <collision>
-      <origin xyz="0 0 0" rpy="0 0 ${pi/2}"/>
+      <origin xyz="0 0 0" rpy="${pi} 0 ${pi/2}"/>
       <geometry>
         <mesh filename="package://iai_daisy_description/meshes/FL-ISO50-WPG300_WITH_FILLET.stl" scale="0.001 0.001 0.001"/>
@@ -175,8 +231,11 @@
     <parent link="right_flange"/>
     <child link="right_gripper_mounting_plate"/>
-    <origin xyz="0 0 0.005" rpy="${pi/2} 0 ${pi/2}"/>
-  </joint>
+    <origin xyz="0.005 0 0" rpy="-${pi/2} 0 -${pi/2}"/>
+  </joint>
+  <!-- === Cable guide on the right gripper === -->
+  <xacro:gripper_side_cylinder parent="right_gripper_mounting_plate" prefix="right_gripper" />
+  <xacro:wrist_collision_cylinder_macro parent="right_wrist_2_link" prefix="right_gripper" />
   <xacro:wsg_300_120_xacro parent="right_gripper_mounting_plate" name="right_gripper">
-    <origin xyz="0 0 0" rpy="0 0 -${pi/2}"/>
+    <origin xyz="0 0 0.005" rpy="0 0 -${pi/2}"/>
   </xacro:wsg_300_120_xacro>
   <link name="left_gripper_left_finger_tip_link">

Commit message: Fix DAiSy URDF/XACRO
Change thickness of one of the adapter mounting
plates from 0.006 to 0.01 like on the real robot.

File: iai_daisy_description/robots/daisy.urdf.xacro (robot description, xacro)
@@ -58,5 +58,5 @@
   <xacro:property name="right_arm_mounting_plate_width" value="0.18" />
   <xacro:property name="right_arm_mounting_plate_length" value="0.15" />
-  <xacro:property name="right_arm_mounting_plate_height" value="0.006" />
+  <xacro:property name="right_arm_mounting_plate_height" value="0.01" />
   <xacro:property name="right_arm_mounting_plate_x_offset" value="0.994" />
   <xacro:property name="right_arm_mounting_plate_y_offset" value="0.368" />
